Commit message: added pick_place code, corrected the readme

File: denso_robot_descriptions/vs060_hand_description/vs060_hand.urdf (robot description, URDF)
Before this commit: robot vs060_hand, 11 links, 10 joints
Joints:
- joint panda_finger_joint2: mimic joint=panda_finger_joint1 -> (none)
- joint panda_hand_joint: origin xyz=0 0 0 rpy=0 0 0.585375 -> xyz=0 0 0.002 rpy=0 0 0.0

Commit message: changed position controller to effort controller

File: denso_robot_descriptions/vs060_hand_description/vs060_hand.urdf (robot description, URDF)
Before this commit: robot vs060_hand, 11 links, 10 joints
Links:
- link J1: mass 1 -> 4.327
- link J2: mass 1 -> 9.475
- link J4: mass 1 -> 1.799
- link J5: mass 1 -> 1.211
- link J6: mass 1 -> 4.154
- link base_link: mass 1 -> 1000
- link panda_hand: mass 1 -> 0.73
- link panda_leftfinger: mass 1 -> 0.1
- link panda_rightfinger: mass 1 -> 0.1
Joints:
- joint joint_1: limit lower=-2.96706 upper=2.96706 effort=1 velocity=3.92699081698724 -> lower=-2.96706 upper=2.96706 effort=19.7336 velocity=0.5
- joint joint_2: limit lower=-2.094395 upper=2.094395 effort=1 velocity=2.61799387799149 -> lower=-2.0944 upper=2.0944 effort=16.8447 velocity=0.5
- joint joint_3: limit lower=-2.181662 upper=2.70526 effort=1 velocity=2.85832571599111 -> lower=-2.18166 upper=2.70526 effort=20.7089 velocity=0.5
- joint joint_4: limit lower=-4.712389 upper=4.712389 effort=1 velocity=3.92699081698724 -> lower=-4.71239 upper=4.71239 effort=20.9665 velocity=0.5
- joint joint_5: limit lower=-2.094395 upper=2.094395 effort=1 velocity=3.02168853397778 -> lower=-2.0944 upper=2.0944 effort=23.7229 velocity=0.5
- joint joint_6: limit lower=-6.283185 upper=6.283185 effort=1 velocity=6.28318530717959 -> lower=-6.28319 upper=6.28319 effort=33.5103 velocity=0.5
